Commit message: 🔧 Add ros2_control mock hardware + rename gripper joint
- Add <ros2_control> tag to URDF with mock_components/GenericSystem
- Add mimic tag on joint_right (mirrors gripper_joint × -1.0)
- Rename joint_left → gripper_joint (single motor drives both fingers)
- Add controllers YAML config for joint_state_broadcaster,
  joint_trajectory_controller, and gripper_controller

File: rebot_description/urdf/rebot_b601_rs.urdf (robot description, URDF)
Before this commit: robot rebot_b601_rs, 11 links, 10 joints
Joints:
- removed joint joint_left
- added joint gripper_joint: type prismatic, parent gripper_end, child gripper_left, origin xyz=-0.041939 -7.3385E-05 0 rpy=1.5708 -1.5708 0, axis 0 0 1, limit lower=0 upper=0.05 effort=500 velocity=10
- joint joint_right: mimic (none) -> joint=gripper_joint multiplier=-1.0 offset=0.0
